File: hardware/pcb/mp3alarm.kicad_pcb (KiCad board)
At the start: 2 copper layers, 67 x 54 mm, 69 parts, among them IC1 RDA5807FP, J1 AUDIO, J10 Conn_Coaxial, J11 USB_C_Receptacle_USB2.0, J2 SW0, J3 SW1, J4 AudioJack3, J5 I2C, J6 TM1637, J7 microSD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

Commit message: Updated PCB
Parts:
- C2: value 1uF -> 22nF
- moved C2 21.3 mm to (84.3, 72.9)
Connections:
- C2 pad 1: GND -> VCC
- C2 pad 2: BOOT -> GND
Routing:
- net BOOT: track 6.29 -> 2.94 mm
- net TM_CLK: track 28.0 -> 28.6 mm
- net GND: vias 51 -> 76
