File: hardware/pcb/mp3alarm.kicad_sch (KiCad schematic)
At the start: 69 parts, among them IC1 RDA5807FP, J1 AUDIO, J10 Conn_Coaxial, J11 USB_C_Receptacle_USB2.0, J2 SW0, J3 SW1, J4 AudioJack3, J5 I2C, J6 TM1637, J7 microSD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

Commit message: Updated PCB
Parts:
- C2: value 1uF -> 22nF
Connections:
- net BOOT: no longer C2.2
- net GND: now also C2.2; no longer C2.1
- net VCC: now also C2.1
Other:
- moved on the sheet: C3, C4, C5, D1, D2, D3, D4, H1, H2, H3, H4, J11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
